Commit message: small success

File: arac_description/urdf/wheel/wheel.urdf.xacro (robot description, xacro)
@@ -37,9 +37,12 @@
     </joint>
     <gazebo reference="${leg}_WH" >
-        <kp>${kp_wheel}</kp>
+    	<kp>${kp_wheel}</kp>
         <kd>${kd_wheel}</kd>
         <mu1>${mu_wheel}</mu1>
         <mu2>${mu_wheel}</mu2>
+        <fdir1 value="1 0 0"/>
         <minDepth> ${wheel_minDepth} </minDepth>
+        <maxVel>100.0</maxVel>
+        <material>Gazebo/Black</material>
     </gazebo>
   </xacro:macro>

File: arac_description/urdf/wheel/wheel_parameters.urdf.xacro (robot description, xacro)
@@ -15,5 +15,5 @@
   <xacro:property name="kp_wheel"            value= "1000000.0" />
   <xacro:property name="kd_wheel"            value= "100.0" />
-  <xacro:property name="mu_wheel"            value= "0.8" />
+  <xacro:property name="mu_wheel"            value= "1" />
   <xacro:property name="wheel_minDepth"      value= "0.001" /> <!-- [m] -->
 </robot>
