Commit message: Hokuyo tarayici eklendi. Bunun test edebilmek icin gazeboya biraz ortam eklemek gerekiyor.

File: arac_description/urdf/arac.urdf.xacro (robot description, xacro)
@@ -43,3 +43,30 @@
     </properties>
   </xacro:wheel>
+    <!-- Hokuyo Laser -->
+    <joint name="hokuyo_joint" type="fixed">
+       <axis xyz="0 1 0" />
+       <origin xyz="0 0 ${h_b}" rpy="0 0 0"/>
+       <parent link="base"/>
+       <child link="hokuyo_link"/>
+    </joint>
+    <!-- Hokuyo Laser -->
+    <link name="hokuyo_link">
+     <collision>
+       <origin xyz="0 0 0" rpy="0 0 0"/>
+       <geometry>
+         <box size="0.1 0.1 0.1"/>
+       </geometry>
+     </collision>
+     <visual>
+       <origin xyz="0 0 0" rpy="0 0 0"/>
+       <geometry>
+         <mesh filename= "package://arac_description/urdf/mesh/hokuyo.dae"/>
+       </geometry>
+     </visual>
+     <inertial>
+       <mass value="1e-5" />
+       <origin xyz="0 0 0" rpy="0 0 0"/>
+       <inertia ixx="1e-6" ixy="0" ixz="0" iyy="1e-6" iyz="0" izz="1e-6" />
+     </inertial>
+    </link>
 </robot>

File: arac_description/urdf/include/arac_utils.urdf.xacro (robot description, xacro)
@@ -3,4 +3,5 @@
   <!-- Import shared components -->
     <xacro:include filename="$(find arac_description)/urdf/include/arac_plugin.gazebo.xacro"/>
+    <xacro:include filename="$(find arac_description)/urdf/include/hokuyo_plugin.gazebo.xacro"/>
   <!-- Math constants -->
   <xacro:property name="PI" value="3.1415926535897931"/>

Commit message: Durum kestirimci eklendi ve yeni bir denetleyici altyapisi olusturuldu

File: arac_description/urdf/arac.urdf.xacro (robot description, xacro)
@@ -70,3 +70,29 @@
      </inertial>
     </link>
+    <!-- Imu Link -->
+    <joint name="imu_joint" type="fixed">
+       <axis xyz="0 1 0" />
+       <origin xyz="0 0 0" rpy="0 0 0"/>
+       <parent link="base"/>
+       <child link="imu_link"/>
+    </joint>
+    <link name="imu_link">
+     <collision>
+       <origin xyz="0 0 0" rpy="0 0 0"/>
+       <geometry>
+         <box size="0.1 0.1 0.1"/>
+       </geometry>
+     </collision>
+     <visual>
+       <origin xyz="0 0 0" rpy="0 0 0"/>
+       <geometry>
+         <box size="0.1 0.1 0.1"/>
+       </geometry>
+     </visual>
+     <inertial>
+       <mass value="1e-5" />
+       <origin xyz="0 0 0" rpy="0 0 0"/>
+       <inertia ixx="1e-6" ixy="0" ixz="0" iyy="1e-6" iyz="0" izz="1e-6" />
+     </inertial>
+    </link>
 </robot>

File: arac_description/urdf/include/arac_utils.urdf.xacro (robot description, xacro)
@@ -4,4 +4,5 @@
     <xacro:include filename="$(find arac_description)/urdf/include/arac_plugin.gazebo.xacro"/>
     <xacro:include filename="$(find arac_description)/urdf/include/hokuyo_plugin.gazebo.xacro"/>
+    <xacro:include filename="$(find arac_description)/urdf/include/imu_plugin.gazebo.xacro"/>
   <!-- Math constants -->
   <xacro:property name="PI" value="3.1415926535897931"/>

File: arac_description/urdf/include/hokuyo_plugin.gazebo.xacro (robot description, xacro)
@@ -37,3 +37,22 @@
     </sensor>
   </gazebo>
+  <gazebo reference="imu_link">
+      <gravity>true</gravity>
+      <sensor name="imu_sensor" type="imu">
+        <always_on>true</always_on>
+        <update_rate>100</update_rate>
+        <visualize>true</visualize>
+        <topic>__default_topic__</topic>
+        <plugin filename="libgazebo_ros_imu_sensor.so" name="imu_plugin">
+          <topicName>imu</topicName>
+          <bodyName>imu_link</bodyName>
+          <updateRateHZ>10.0</updateRateHZ>
+          <gaussianNoise>0.0</gaussianNoise>
+          <xyzOffset>0 0 0</xyzOffset>
+          <rpyOffset>0 0 0</rpyOffset>
+          <frameName>imu_link</frameName>
+        </plugin>
+        <pose>0 0 0 0 0 0</pose>
+      </sensor>
+    </gazebo>
 </robot>

File: arac_description/urdf/wheel/wheel_parameters.urdf.xacro (robot description, xacro)
@@ -3,14 +3,14 @@
   <xacro:property name="r_wheel"                value= "0.15"/> <!-- [m] -->
   <xacro:property name="w_wheel"                value= "0.02"/> <!-- [m] -->
-  <xacro:property name="m_wheel"                value= "10.0"/> <!-- [kg] -->
+  <xacro:property name="m_wheel"                value= "0.5"/> <!-- [kg] -->
   <xacro:property name="x_wheel"                value= "0.2"/> <!-- m -->
   <xacro:property name="y_wheel"                value= "0.2"/> <!-- m -->
   <xacro:property name="z_wheel"                value= "-0.05"/> <!-- m -->
-  <xacro:property name="B_Ixx_wheel"            value= "0.01"/> <!-- [kg * m^2] -->
-  <xacro:property name="B_Iyy_wheel"            value= "0.1000"/> <!-- [kg * m^2] -->
+  <xacro:property name="B_Ixx_wheel"            value= "0.0100"/> <!-- [kg * m^2] -->
+  <xacro:property name="B_Iyy_wheel"            value= "0.0100"/> <!-- [kg * m^2] -->
   <xacro:property name="B_Izz_wheel"            value= "0.1000"/> <!-- [kg * m^2] -->
   <xacro:property name="B_Ixy_wheel"            value= "0.0000"/> <!-- [kg * m^2] -->
-  <xacro:property name="B_Ixz_wheel"            value="-0.0000"/> <!-- [kg * m^2] -->
-  <xacro:property name="B_Iyz_wheel"            value="-0.000"/> <!-- [kg * m^2] -->
+  <xacro:property name="B_Ixz_wheel"            value= "0.0000"/> <!-- [kg * m^2] -->
+  <xacro:property name="B_Iyz_wheel"            value= "0.000"/> <!-- [kg * m^2] -->
   <xacro:property name="kp_wheel"            value= "1000000.0" />
   <xacro:property name="kd_wheel"            value= "100.0" />
